Commit message: Refactor robot_core.xacro: clean up formatting, remove unnecessary attributes, and ensure consistent geometry definitions

File: description/robot_core.xacro (robot description, xacro)
@@ -1,7 +1,7 @@
 <?xml version="1.0"?>
-<robot xmlns:xacro="http://www.ros.org/wiki/xacro"  name="robot">
-  <xacro:include filename="inertial_macros.xacro" />
+<robot xmlns:xacro="http://www.ros.org/wiki/xacro" >
+  <xacro:include filename="inertial_macros.xacro"/>
   <material name="white">
-    <color rgba="1 1 1 1"/>
+    <color rgba="1 1 1 1" />
   </material>
   <material name="orange">
@@ -16,5 +16,6 @@
   <!-- BASE LINK -->
   <link name="base_link">
-  </link>
+    </link>
+  <!-- CHASSIS LINK -->
   <joint name="chassis_joint" type="fixed">
     <parent link="base_link"/>
@@ -22,8 +23,7 @@
     <origin xyz="-0.1 0 0"/>
   </joint>
-  <!-- CHASSIS-->
   <link name="chassis">
     <visual>
-      <origin xyz="0.15 0 0.075" rpy="0 0 0"/>
+      <origin xyz="0.15 0 0.075"/>
       <geometry>
         <box size="0.3 0.3 0.15"/>
@@ -32,47 +32,41 @@
     </visual>
     <collision>
-      <origin xyz="0.15 0 0.075" rpy="0 0 0"/>
+      <origin xyz="0.15 0 0.075"/>
       <geometry>
         <box size="0.3 0.3 0.15"/>
       </geometry>
-      <material name="white"/>
     </collision>
-        <xacro:inertial_box mass="0.5" x="0.3" y="0.3" z="0.15">
+    <xacro:inertial_box mass="0.5" x="0.3" y="0.3" z="0.15">
       <origin xyz="0.15 0 0.075" rpy="0 0 0"/>
     </xacro:inertial_box>
   </link>
-  <!-- LEFT WHEEL -->
+  <!-- LEFT WHEEL LINK -->
   <joint name="left_wheel_joint" type="continuous">
     <parent link="base_link"/>
     <child link="left_wheel"/>
-    <origin xyz="0 0.175 0" rpy="-${pi/2} 0 0"/>
+    <origin xyz="0 0.175 0" rpy="-${pi/2} 0 0" />
     <axis xyz="0 0 1"/>
-    <xacro:inertial_cylinder mass="0.1" length="0.05" radius="0.05">
-      <origin xyz="0 0 0" rpy="0 0 0"/>
-    </xacro:inertial_cylinder>
   </joint>
   <link name="left_wheel">
     <visual>
       <geometry>
-        <cylinder length="0.04" radius="0.05" />
+        <cylinder radius="0.05" length="0.04"/>
       </geometry>
       <material name="blue"/>
     </visual>
     <collision>
-        <!-- <origin xyz="0 0 0" rpy="0 0 0"/> -->
       <geometry>
-        <cylinder length="0.04" radius="0.05" />
+        <cylinder radius="0.05" length="0.04"/>
       </geometry>
-      <material name="blue"/>
     </collision>
-        <xacro:inertial_cylinder mass="0.1" length="0.04" radius="0.05">
+    <xacro:inertial_cylinder mass="0.1" length="0.04" radius="0.05">
       <origin xyz="0 0 0" rpy="0 0 0"/>
     </xacro:inertial_cylinder>
   </link>
-  <!-- RIGHT WHEEL -->
+  <!-- RIGHT WHEEL LINK -->
   <joint name="right_wheel_joint" type="continuous">
     <parent link="base_link"/>
     <child link="right_wheel"/>
-    <origin xyz="0 -0.175 0" rpy="${pi/2} 0 0"/>
+    <origin xyz="0 -0.175 0" rpy="${pi/2} 0 0" />
     <axis xyz="0 0 -1"/>
   </joint>
@@ -80,29 +74,27 @@
     <visual>
       <geometry>
-        <cylinder length="0.04" radius="0.05" />
+        <cylinder radius="0.05" length="0.04"/>
       </geometry>
       <material name="blue"/>
     </visual>
     <collision>
-      <!-- <origin xyz="0 0 0" rpy="0 0 0"/> -->
       <geometry>
-        <cylinder length="0.04" radius="0.05" />
+        <cylinder radius="0.05" length="0.04"/>
       </geometry>
-      <material name="blue"/>
     </collision>
-        <xacro:inertial_cylinder mass="0.1" length="0.04" radius="0.05">
+    <xacro:inertial_cylinder mass="0.1" length="0.04" radius="0.05">
       <origin xyz="0 0 0" rpy="0 0 0"/>
     </xacro:inertial_cylinder>
   </link>
-  <!-- CASTER WHEEL -->
+  <!-- CASTER WHEEL LINK -->
   <joint name="caster_wheel_joint" type="fixed">
     <parent link="chassis"/>
     <child link="caster_wheel"/>
-    <origin xyz="0.24 0 0" rpy="0 0 0"/>
+    <origin xyz="0.24 0 0"/>
   </joint>
   <link name="caster_wheel">
     <visual>
       <geometry>
-        <sphere radius="0.05" />
+        <sphere radius="0.05"/>
       </geometry>
       <material name="black"/>
@@ -110,11 +102,10 @@
     <collision>
       <geometry>
-        <sphere radius="0.05" />
+        <sphere radius="0.05"/>
       </geometry>
-      <material name="black"/>
     </collision>
-        <xacro:inertial_cylinder mass="0.1" length="0.04" radius="0.05">
+    <xacro:inertial_sphere mass="0.1" radius="0.05">
       <origin xyz="0 0 0" rpy="0 0 0"/>
-    </xacro:inertial_cylinder>
+    </xacro:inertial_sphere>
   </link>
 </robot>

Commit message: Update README.md with terminal commands and add view_robot.rviz configuration for RViz visualization

File: description/robot_core.xacro (robot description, xacro)
@@ -59,4 +59,5 @@
         <cylinder radius="0.05" length="0.04"/>
       </geometry>
+      <material name="blue"/>
     </collision>
     <xacro:inertial_cylinder mass="0.1" length="0.04" radius="0.05">
@@ -81,4 +82,5 @@
       <geometry>
         <cylinder radius="0.05" length="0.04"/>
+        <material name="blue"/>
       </geometry>
     </collision>
@@ -103,4 +105,5 @@
       <geometry>
         <sphere radius="0.05"/>
+        <material name="black"/>
       </geometry>
     </collision>

Commit message: Add Gazebo control and simulation launch files; update robot description

File: description/robot_core.xacro (robot description, xacro)
@@ -17,5 +17,5 @@
   <link name="base_link">
     </link>
-  <!-- CHASSIS LINK -->
+  <!-- CHASSIS Joint -->
   <joint name="chassis_joint" type="fixed">
     <parent link="base_link"/>
@@ -23,4 +23,5 @@
     <origin xyz="-0.1 0 0"/>
   </joint>
+  <!-- CHASSIS LINK DEFINITION -->
   <link name="chassis">
     <visual>
@@ -41,5 +42,8 @@
     </xacro:inertial_box>
   </link>
-  <!-- LEFT WHEEL LINK -->
+    <gazebo reference="chassis">
+        <material>Gazebo/Orange</material>
+    </gazebo>
+  <!-- LEFT WHEEL Joint -->
   <joint name="left_wheel_joint" type="continuous">
     <parent link="base_link"/>
@@ -48,4 +52,5 @@
     <axis xyz="0 0 1"/>
   </joint>
+  <!-- LEFT WHEEL LINK -->
   <link name="left_wheel">
     <visual>
@@ -59,5 +64,4 @@
         <cylinder radius="0.05" length="0.04"/>
       </geometry>
-      <material name="blue"/>
     </collision>
     <xacro:inertial_cylinder mass="0.1" length="0.04" radius="0.05">
@@ -65,4 +69,7 @@
     </xacro:inertial_cylinder>
   </link>
+    <gazebo reference="left_wheel">
+        <material>Gazebo/Blue</material>
+    </gazebo>
   <!-- RIGHT WHEEL LINK -->
   <joint name="right_wheel_joint" type="continuous">
@@ -82,5 +89,4 @@
       <geometry>
         <cylinder radius="0.05" length="0.04"/>
-        <material name="blue"/>
       </geometry>
     </collision>
@@ -89,4 +95,7 @@
     </xacro:inertial_cylinder>
   </link>
+    <gazebo reference="right_wheel">
+        <material>Gazebo/Blue</material>
+    </gazebo>
   <!-- CASTER WHEEL LINK -->
   <joint name="caster_wheel_joint" type="fixed">
@@ -105,5 +114,4 @@
       <geometry>
         <sphere radius="0.05"/>
-        <material name="black"/>
       </geometry>
     </collision>
@@ -112,3 +120,8 @@
     </xacro:inertial_sphere>
   </link>
+ <gazebo reference="caster_wheel">
+        <material>Gazebo/White</material>
+        <mu1 value="0.001"/>
+        <mu2 value="0.001"/>
+    </gazebo>
 </robot>

Commit message: Add camera and lidar descriptions; include in robot.urdf.xacro
Integrates camera and LiDAR into robot model

Adds dedicated Xacro descriptions for a camera and a LiDAR sensor. These definitions include physical links, visual properties, and Gazebo sensor plugins for each.

The camera setup incorporates an optical frame to ensure correct ROS topic orientation. The LiDAR includes complete collision and inertial properties for accurate simulation.

These new sensor components are included in the main robot URDF Xacro file, enabling the robot to perceive its environment in simulation. A 'red' material is also added for sensor visualization.

File: description/robot_core.xacro (robot description, xacro)
@@ -13,4 +13,7 @@
   <material name="black">
     <color rgba="0 0 0 1"/>
+  </material>
+  <material name="red">
+      <color rgba="1 0 0 1"/>
   </material>
   <!-- BASE LINK -->
