Commit message: Enhance wheel creation macro to accept joint names for better customization

File: description/common_macros.xacro (robot description, xacro)
@@ -1,5 +1,6 @@
 <?xml version="1.0"?>
 <robot xmlns:xacro="http://www.ros.org/wiki/xacro">
-    <xacro:macro name="create_wheel" params="name x_offset y_offset">
+    <xacro:macro name="create_wheel" params="name x_offset y_offset joint_name:=''">
+        <xacro:property name="joint_id" value="${joint_name if joint_name != '' else name + '_joint'}" />
         <link name="${name}">
             <visual>
@@ -21,5 +22,5 @@
             </inertial>
         </link>
-        <joint name="${name}_joint" type="continuous">
+        <joint name="${joint_id}" type="continuous">
             <parent link="chassis"/>
             <child link="${name}"/>

File: description/robot_core.xacro (robot description, xacro)
@@ -1,4 +1,4 @@
 <?xml version="1.0"?>
-<robot xmlns:xacro="http://www.ros.org/wiki/xacro" >
+<robot xmlns:xacro="http://www.ros.org/wiki/xacro">
     <xacro:include filename="inertial_macros.xacro"/>
     <xacro:include filename="common_macros.xacro"/>
@@ -45,5 +45,5 @@
     </link>
     <!-- CHASSIS LINK -->
-<!--
+    <!--
     <joint name="chassis_joint" type="fixed">
         <parent link="base_link"/>
@@ -103,5 +103,5 @@
     </gazebo>
     <!-- LEFT WHEEL LINK -->
-<!--
+    <!--
     <joint name="left_wheel_joint" type="continuous">
         <parent link="base_link"/>
@@ -153,8 +153,12 @@
     <gazebo reference="right_wheel">
         <material>Gazebo/Blue</material></gazebo> -->
-    <xacro:create_wheel name="front_left_wheel"  x_offset="${wheel_offset_x}" y_offset="${wheel_offset_y}"/>
-    <xacro:create_wheel name="front_right_wheel" x_offset="${wheel_offset_x}" y_offset="-${wheel_offset_y}"/>
-    <xacro:create_wheel name="rear_left_wheel"   x_offset="-${wheel_offset_x}" y_offset="${wheel_offset_y}"/>
-    <xacro:create_wheel name="rear_right_wheel"  x_offset="-${wheel_offset_x}" y_offset="-${wheel_offset_y}"/>
+    <xacro:create_wheel name="front_left_wheel" joint_name="front_left_wheel_joint" x_offset="${wheel_offset_x}" y_offset="${wheel_offset_y}"/>
+    <xacro:create_wheel name="front_right_wheel" joint_name="front_right_wheel_joint" x_offset="${wheel_offset_x}" y_offset="-${wheel_offset_y}"/>
+    <xacro:create_wheel name="rear_left_wheel" joint_name="rear_left_wheel_joint" x_offset="-${wheel_offset_x}" y_offset="${wheel_offset_y}"/>
+    <xacro:create_wheel name="rear_right_wheel" joint_name="rear_right_wheel_joint" x_offset="-${wheel_offset_x}" y_offset="-${wheel_offset_y}"/>
+    <!-- <xacro:create_wheel name="front_left_wheel" x_offset="${wheel_offset_x}" y_offset="${wheel_offset_y}"/>
+<xacro:create_wheel name="front_right_wheel" x_offset="${wheel_offset_x}" y_offset="-${wheel_offset_y}"/>
+<xacro:create_wheel name="rear_left_wheel" x_offset="-${wheel_offset_x}" y_offset="${wheel_offset_y}"/>
+<xacro:create_wheel name="rear_right_wheel" x_offset="-${wheel_offset_x}" y_offset="-${wheel_offset_y}"/> -->
     <!-- CASTER WHEEL LINK -->
     <!-- <joint name="caster_wheel_joint" type="fixed">
